Commit message: Phase 3.5 — L2 하드웨어 정합 + 회귀 하네스 결함 2건 수정 (§9.1)
시뮬 라이다를 L2 공칭으로 전환하고, L1 전제로 유도된 파라미터를 전수
재유도한다. 계획 v3.1.1 §1.1~1.4 · §6.1~6.6 · §9.1.

센서 (§6.6)
· lidar_4D_lidar.xacro 를 lidar_gen:=l1|l2 인자화 (기본 l2)
  5.55Hz / min 0.05m / 480×24 ≈ 63,936 pts/s (데이터시트 유효 64,000 근사)
  l1 값은 v2 재현용으로 보존 — launch 에 동일 인자 노출

재유도 (§6.1~6.4)
· emergency/blind_hold_clearance 0.60→0.30
  사각의 실효 경계가 센서 min_range(0.8)에서 ROI 크롭(roi_x_min 0.5)으로
  이동 — 유도식의 입력 심볼이 교체된 경우. 구조적 동형 유지
  (v2 0.95≥0.8+0.15 ↔ v3 0.65≥0.5+0.15). head_on·static_stop N≥5 로 유효화
· T_frame 0.10→0.18 파급: publish_rate 5.55 · assoc_max_dist 2.2 ·
  sensor_timeout 0.9 · cvm_latency_max 0.5 · vel_max_dt 0.8
  vel_max_dt 는 v2 잠재 결함이기도 하다 — 코스팅 상한 직후 재연관 시
  dtm 0.72s 가 상한 0.5를 넘어 속도 갱신이 조용히 스킵됐다
· self box x ∓0.40→∓0.45 (시뮬 판) — L2 에서 이 박스가 1차 방어선이 된다

열화 프로파일 (§6.5)
· real_l2 / worst_case_l2 신설, 구판 2종 DEPRECATED
· real_l2 의 keep 1.0 이 핵심: real_l1 의 0.20은 시뮬 균일 링을 L1 유효율로
  깎는 계수였다 — 시뮬이 L2 공칭으로 내려온 지금 얹으면 이중 열화

회귀 하네스 결함 2건 (재기준화 중 발견, L2 무관 — v2 수치에도 소급)
· kill_gazebo_leftovers 가 gz/bridge 만 죽여 파이썬 노드가 살아남음.
  유령 노드 34분 생존 실측 — 같은 ROS 그래프에 계속 발행해 판정을 오염
  (오염 시 static_stop travel 0.00m/ESTOP, 변경 전 대조군도 stops=145).
  LEFTOVER_PATTERNS 로 스택 전체 종료
· base 월드에 RTF 캡이 없어 머신이 한가하면 RTF 0.50 → 요구 벽시계 렌더율이
  GPU 라이다 상한(~2.5Hz)을 넘어 심시간 주기 붕괴(0.72~0.90s).
  A/B: 캡 O → PASS(SLOW_DOWN 진입, 0.409m) / 캡 X → FAIL(미진입, 0.316m 스침).
  RTF 캡은 성능 편의가 아니라 게이트 성립 조건 — worlds.py 가 주입

대장 (§4.3)
· sensor_generation: L1 레코드 잔여 0. 신규 4종 등재 (sim_lidar_config,
  degrade_profile, sensor_timeout, publish_rate)
· roi_x_max 는 값 유지 — §1.4 재유도 필요 17.6m > 가용 15m 구속은 미해소,
  해소 수단은 v_robot_max 하향(§1.4 ③). note 에 명시

pytest 187/187. 델타 문서: docs/changelog/l1_to_l2_delta.md

Co-Authored-By: Claude Opus 5 (1M context) <noreply@anthropic.com>

File: ros2_ws/src/unitree_go2_ros2/unitree_go2_description/urdf/lidar_4D_lidar.xacro (robot description, xacro)
@@ -33,12 +33,26 @@
         <origin rpy="2.879 0.0 1.5705" xyz="0.25 -0.038 -0.03"/>
     </joint>
+    <!-- 센서 세대 스위치 (Phase 3.5, 계획 v3.1.1 §6.6): 기본 l2.
+         L1↔L2 델타 재현(l1_to_l2_delta.md)용으로 lidar_gen:=l1 을 남긴다.
+         l1 값(10 Hz / 0.8~30 m / 600×30)은 v2 시뮬 설정 보존용 — 0.8 m는
+         URDF 설정값이지 L1 데이터시트 블라인드가 아님 (§1.2 v3.1 정정).
+         l2 값: 수평 5.55 Hz, 근거리 0.05 m, 480×24×5.55 ≈ 63,936 pts/s
+         ≈ 유효 64,000 pts/s (데이터시트, PROVISIONAL — 측정 5로 확정).
+         비반복 스캔·반사율 dropout·밀도 불균일은 gz 라이다로 표현 불가 →
+         degrade 노드 real_l2 프로파일 담당 (§6.5). -->
+    <xacro:arg name="lidar_gen" default="l2"/>
+    <xacro:property name="lidar_gen_v" value="$(arg lidar_gen)"/>
+    <xacro:property name="lidar_rate" value="${10 if lidar_gen_v == 'l1' else 5.55}"/>
+    <xacro:property name="lidar_h_samples" value="${600 if lidar_gen_v == 'l1' else 480}"/>
+    <xacro:property name="lidar_v_samples" value="${30 if lidar_gen_v == 'l1' else 24}"/>
+    <xacro:property name="lidar_min_range" value="${0.8 if lidar_gen_v == 'l1' else 0.05}"/>
     <gazebo reference="lidar_l1_link">
         <sensor name="lidar_l1" type="gpu_lidar">
             <topic>unitree_lidar</topic>
-            <update_rate>10</update_rate>
+            <update_rate>${lidar_rate}</update_rate>
             <lidar>
                 <scan>
                     <horizontal>
-                        <samples>600</samples>
+                        <samples>${lidar_h_samples}</samples>
                         <resolution>1</resolution>
                         <min_angle>-3.14159</min_angle>
@@ -46,5 +60,5 @@
                     </horizontal>
                     <vertical>
-                        <samples>30</samples>
+                        <samples>${lidar_v_samples}</samples>
                         <resolution>1</resolution>
                         <min_angle>-0.785398</min_angle>
@@ -53,5 +67,5 @@
                 </scan>
                 <range>
-                    <min>0.8</min>
+                    <min>${lidar_min_range}</min>
                     <max>30.0</max>
                     <resolution>0.001</resolution>
