Commit message: Phase 0: 실기체 센서 구성 정합 — D435i RGBD+IMU 추가, Velodyne 제거
- RGB 카메라 → D435i rgbd_camera (hfov 87°, depth 0.105~10m, IMU 200Hz)
- Velodyne 미탑재 실기체에 맞춰 include 제거, L1(/unitree_lidar/points)만 유지
- trunk collision 이름 명시(trunk_collision), rviz 카메라/포인트클라우드 표시 갱신

Co-Authored-By: Claude Fable 5 <noreply@anthropic.com>

File: ros2_ws/src/go2_simulation/urdf/unitree_go2_gazebo.xacro (robot description, xacro)
@@ -115,16 +115,16 @@
     </sensor>
   </gazebo>-->
-  <!-- Camera Plugin with physical calibration profile -->
+  <!-- RealSense D435i RGBD Camera + IMU (실제 하드웨어 매칭) -->
   <gazebo reference="camera_link">
-    <sensor name="rgb_camera" type="camera">
+    <sensor name="rgbd_camera" type="rgbd_camera">
       <pose>0 0 0 0 0 0</pose>
-      <update_rate>30</update_rate>
+      <update_rate>15</update_rate>
       <always_on>1</always_on>
-      <visualize>1</visualize>
-      <topic>rgb_image</topic>
+      <visualize>0</visualize>
+      <topic>d435i</topic>
       <gz_frame_id>camera_link</gz_frame_id>
       <camera>
-        <!-- fx=542.4, width=640 -> hfov = 2*arctan(640/(2*542.4)) ≈ 1.066 rad -->
-        <horizontal_fov>1.066</horizontal_fov>
+        <!-- D435i RGB: hfov ~87 deg = 1.518 rad -->
+        <horizontal_fov>1.518</horizontal_fov>
         <image>
           <width>640</width>
@@ -132,19 +132,34 @@
           <format>R8G8B8</format>
         </image>
+        <depth_camera>
+          <clip>
+            <near>0.105</near>
+            <far>10.0</far>
+          </clip>
+        </depth_camera>
         <clip>
           <near>0.05</near>
           <far>20.0</far>
         </clip>
-        <!-- Distortion parameters from cali_result.txt -->
-        <!-- dist: [k1, k2, p1, p2, k3] -->
-        <distortion>
-          <k1>-0.524518908</k1>
-          <k2>0.369148040</k2>
-          <k3>-0.172802932</k3>
-          <p1>0.002309632</p1>
-          <p2>0.000172606</p2>
-          <center>0.5 0.5</center>
-        </distortion>
       </camera>
+    </sensor>
+    <!-- D435i 내장 IMU (BMI055) -->
+    <sensor name="d435i_imu" type="imu">
+      <always_on>true</always_on>
+      <update_rate>200</update_rate>
+      <topic>d435i/imu</topic>
+      <gz_frame_id>camera_link</gz_frame_id>
+      <imu>
+        <angular_velocity>
+          <x><noise type="gaussian"><mean>0.0</mean><stddev>1e-3</stddev></noise></x>
+          <y><noise type="gaussian"><mean>0.0</mean><stddev>1e-3</stddev></noise></y>
+          <z><noise type="gaussian"><mean>0.0</mean><stddev>1e-3</stddev></noise></z>
+        </angular_velocity>
+        <linear_acceleration>
+          <x><noise type="gaussian"><mean>0.0</mean><stddev>2e-2</stddev></noise></x>
+          <y><noise type="gaussian"><mean>0.0</mean><stddev>2e-2</stddev></noise></y>
+          <z><noise type="gaussian"><mean>0.0</mean><stddev>2e-2</stddev></noise></z>
+        </linear_acceleration>
+      </imu>
     </sensor>
   </gazebo>

File: ros2_ws/src/go2_simulation/urdf/unitree_go2_robot.xacro (robot description, xacro)
@@ -9,5 +9,5 @@
     <xacro:include filename="$(find go2_simulation)/urdf/unitree_go2_gazebo.xacro"/>
     <!-- <xacro:include filename="$(find unitree_go2_description)/launch/stairs.urdf.xacro"/> -->
-    <xacro:include filename="$(find unitree_go2_description)/urdf/velodyne.xacro"/>
+    <!-- <xacro:include filename="$(find unitree_go2_description)/urdf/velodyne.xacro"/> -->
     <xacro:include filename="$(find unitree_go2_description)/urdf/lidar_4D_lidar.xacro"/>
     <!-- <xacro:stairs stairs="15" xpos="0" ypos="0" zpos="0" /> -->
@@ -43,5 +43,5 @@
             </geometry>
         </visual>
-        <collision>
+        <collision name="trunk_collision">
             <origin rpy="0 0 0" xyz="0 0 0"/>
             <geometry>

Commit message: 눈높이 POV 카메라 추가 — 형상 없는 링크, 기본 OFF 토글
지상 ~1.6m 전방 수평 카메라를 /head_cam/image 로 노출한다.

- head_cam_link: visual/collision 미정의로 Gazebo/RViz에 형상이 없다.
  z=1.375 = 1.6(눈높이) - 0.225(nominal_height). mass는 fixed joint
  lumping 시 trunk 관성에 m*d^2로 더해지므로 1e-5 (trunk_ixx의 0.08%).
  기존 camera_link처럼 1e-3을 쓰면 7.7%로 롤 동역학이 바뀐다.
- head_cam 센서: 640x480@30, FOV 80도. 리드백 27.6MB/s로 기존
  d435i_color(720p@15, 41.5MB/s)보다 가볍지만 렌더 스레드를 L1
  라이다와 공유하므로 head_cam_enabled 기본 false.
- launch 3종에 인자 선언/xacro 전달/브리지 추가. 브리지는 무조건
  등록한다 — 센서 OFF면 데이터만 안 흐르고 무해하다.
  launch.py/TI.py는 기존에 xacro 인자를 넘기지 않았으므로
  cameras_enabled는 건드리지 않아 기존 동작이 불변이다.

Co-Authored-By: Claude Opus 5 (1M context) <noreply@anthropic.com>

File: ros2_ws/src/go2_simulation/urdf/unitree_go2_gazebo.xacro (robot description, xacro)
@@ -197,4 +197,33 @@
   </gazebo>
   </xacro:if>
+  <!-- 눈높이 POV 카메라 (지상 ~1.6m, 전방 수평). 형상 없는 head_cam_link에 부착.
+       640x480@30 = 27.6MB/s 리드백으로 위 d435i_color(720p@15, 41.5MB/s)보다 가볍지만,
+       렌더 스레드는 L1 라이다와 공유하므로 기본 OFF — 데모/POV 때만 켠다. -->
+  <xacro:arg name="head_cam_enabled" default="false"/>
+  <xacro:if value="$(arg head_cam_enabled)">
+  <gazebo reference="head_cam_link">
+    <sensor name="head_cam" type="camera">
+      <pose>0 0 0 0 0 0</pose>
+      <update_rate>30</update_rate>
+      <always_on>1</always_on>
+      <visualize>0</visualize>
+      <topic>head_cam/image</topic>
+      <gz_frame_id>head_cam_link</gz_frame_id>
+      <camera>
+        <!-- 80 deg = 1.396 rad (사람 시야에 가까운 광각) -->
+        <horizontal_fov>1.396</horizontal_fov>
+        <image>
+          <width>640</width>
+          <height>480</height>
+          <format>R8G8B8</format>
+        </image>
+        <clip>
+          <near>0.05</near>
+          <far>200.0</far>
+        </clip>
+      </camera>
+    </sensor>
+  </gazebo>
+  </xacro:if>
   <!-- Main body -->
   <gazebo reference="trunk">

File: ros2_ws/src/go2_simulation/urdf/unitree_go2_robot.xacro (robot description, xacro)
@@ -107,4 +107,20 @@
         <origin rpy="0 -0.05 0" xyz="0.34 0 0.06"/>
     </joint>
+    <!-- 눈높이 POV 카메라 링크 (visual/collision 미정의 = Gazebo/RViz에 형상 없음).
+         z = 1.6(사람 눈높이) - 0.225(nominal_height, trunk 원점 지상고).
+         mass는 fixed joint lumping 시 trunk 관성에 m*d^2로 더해지므로 1e-5로 둔다
+         (1e-5*1.375^2 = trunk_ixx 0.02448의 0.08%). -->
+    <link name="head_cam_link">
+        <inertial>
+            <mass value="1e-5"/>
+            <origin rpy="0 0 0" xyz="0 0 0"/>
+            <inertia ixx="1e-9" ixy="0" ixz="0" iyy="1e-9" iyz="0" izz="1e-9"/>
+        </inertial>
+    </link>
+    <joint name="head_cam_joint" type="fixed">
+        <parent link="trunk"/>
+        <child link="head_cam_link"/>
+        <origin rpy="0 0 0" xyz="0 0 1.375"/>
+    </joint>
     <!-- <joint name="lidar_l1_joint" type="fixed">
         <parent link="base_link"/>
